File: Hardware/Qwiic_RFID_Tag_C/Qwiic_RFID_Tag_C.brd (EAGLE design)
At the start: 25.4 x 25.4 mm, 38 parts, among them J1 Qwiic, J2 Qwiic, U1 ST25DV64KC

Commit message: Update aesthetics
Add SFE logo
Update version number
Change schematic frame to correct version
Update design attribution
Parts:
- removed FRAME1: FRAME-LETTERNO_PACKAGE, SparkFun-Aesthetics:DUMMY
- added FRAME2: FRAME-LETTER, SparkFun-Aesthetics:CREATIVE_COMMONS
- added LOGO2: SFE_LOGO_NAME_FLAME.1_INCH, SparkFun-Aesthetics:SFE_LOGO_NAME_FLAME_.1
- moved U$10 1.02 mm to (12.7, 16.8)
- moved U$11 1.02 mm to (12.7, 16.8)
- moved U$13 1.02 mm to (12.7, 18.8)
- moved U$24 1.02 mm to (12.7, 18.8)
Other:
- board text added: "Revised by: Dryw Wade"
- board text added: "Ricardo Ramos"
Changed lines of the file:
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@@
 <drawing>
 <settings>
-<setting alwaysvectorfont="yes"/>
+<setting alwaysvectorfont="no"/>
 <setting verticaltext="up"/>
 </settings>
@@
 <dimension x1="0" y1="0" x2="0" y2="8.89" x3="-5.08" y3="4.445" textsize="1.778" textratio="15" layer="47" unit="inch"/>
 <dimension x1="0" y1="0" x2="0" y2="25.4" x3="-8.89" y3="12.7" textsize="1.778" textratio="15" layer="47" unit="inch"/>
+<text x="16.51" y="-29.21" size="1.778" layer="51" font="vector">Ricardo Ramos</text>
+<text x="2.54" y="-31.75" size="1.778" layer="51" font="vector">Revised by: Dryw Wade</text>
 </plain>
 <attributes>
@@
 <attribute name="VALUE" x="17.78" y="10.16" size="0.6096" layer="27" font="vector" ratio="20" rot="R180" align="top-center"/>
 </element>
-<element name="FRAME1" library="SparkFun-Aesthetics" package="DUMMY" value="FRAME-LETTERNO_PACKAGE" x="0" y="0" smashed="yes">
-<attribute name="DESIGNER" value="Ricardo Ramos" x="33.02" y="-38.1" size="1.778" layer="27" display="off"/>
-<attribute name="REV" value="X02" x="0" y="0" size="1.778" layer="27" display="off"/>
-<attribute name="VERSION" value="x01" x="33.02" y="-38.1" size="1.778" layer="27" display="off"/>
-</element>
 <element name="J1" library="SparkFun-Connectors" package="JST04_1MM_RA" value="Qwiic" x="20.32" y="8.89" smashed="yes" rot="R90">
 <attribute name="NAME" x="22.479" y="7.493" size="0.6096" layer="25" font="vector" ratio="20" rot="R90"/>
@@
 <element name="U$22" library="output" package="##GPO##8" value="" x="16.51" y="1.778" smashed="yes" rot="MR90"/>
 <element name="U$23" library="output" package="#VEH#7" value="" x="19.05" y="1.778" smashed="yes" rot="MR90"/>
-<element name="U$13" library="SER" package="ST25DV64KC5984" value="" x="12.7" y="19.812" smashed="yes"/>
-<element name="U$24" library="SER" package="ST25DV64KC5984" value="" x="12.7" y="19.812" smashed="yes" rot="MR0"/>
-<element name="U$10" library="output" package="DYNAMIC_RFID_TAG0" value="" x="12.7" y="17.78" smashed="yes"/>
-<element name="U$11" library="output" package="DYNAMIC_RFID_TAG0" value="" x="12.7" y="17.78" smashed="yes" rot="MR0"/>
+<element name="U$13" library="SER" package="ST25DV64KC5984" value="" x="12.7" y="18.796" smashed="yes"/>
+<element name="U$24" library="SER" package="ST25DV64KC5984" value="" x="12.7" y="18.796" smashed="yes" rot="MR0"/>
+<element name="U$10" library="output" package="DYNAMIC_RFID_TAG0" value="" x="12.7" y="16.764" smashed="yes"/>
+<element name="U$11" library="output" package="DYNAMIC_RFID_TAG0" value="" x="12.7" y="16.764" smashed="yes" rot="MR0"/>
 <element name="U$1" library="output" package="#I2C#0" value="" x="6.985" y="8.89" smashed="yes" rot="MR0"/>
+<element name="FRAME2" library="SparkFun-Aesthetics" package="CREATIVE_COMMONS" value="FRAME-LETTER" x="-10.16" y="-29.21" smashed="yes">
+<attribute name="DESIGNER" value="" x="-10.16" y="-29.21" size="1.778" layer="27" display="off"/>
+<attribute name="REV" value="" x="-10.16" y="-29.21" size="1.778" layer="27" display="off"/>
+</element>
+<element name="LOGO2" library="SparkFun-Aesthetics" package="SFE_LOGO_NAME_FLAME_.1" value="SFE_LOGO_NAME_FLAME.1_INCH" x="12.7" y="21.336" smashed="yes"/>
 </elements>
 <signals>

Commit message: Design review updates
All scehmatics:
Change IC text to “Dynamic RFID Tag - ST25DV64KC”
Move decoupling capacitor near IC
Update I2C jumper text to say "traces" instead of "trace"

Version A board:
Fix stray via diameter
Approve jumper overlap error

Version C board:
Add SFE logo to bottom silk
Parts:
- added LOGO4: SFE_LOGO_NAME_FLAME.1_INCH, SparkFun-Aesthetics:SFE_LOGO_NAME_FLAME_.1
Changed lines of the file:
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@@
 </element>
 <element name="LOGO2" library="SparkFun-Aesthetics" package="SFE_LOGO_NAME_FLAME_.1" value="SFE_LOGO_NAME_FLAME.1_INCH" x="12.7" y="21.336" smashed="yes"/>
+<element name="LOGO4" library="SparkFun-Aesthetics" package="SFE_LOGO_NAME_FLAME_.1" value="SFE_LOGO_NAME_FLAME.1_INCH" x="12.7" y="21.336" smashed="yes" rot="MR0"/>
 </elements>
 <signals>

Commit message: Design review updates
Add version letter to silk
Add I2C addresses to schematic
Change PTH silk labels from "3.3V" to "3V3"
Parts:
- removed U$19: (no value), output:#3#3V#0
- added U$2: (no value), output:VERSION_C0
- added U$3: (no value), output:#3V3#0
Changed lines of the file:
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@@
 <drawing>
 <settings>
-<setting alwaysvectorfont="no"/>
+<setting alwaysvectorfont="yes"/>
 <setting verticaltext="up"/>
 </settings>
@@
 <element name="U$17" library="output" package="#LED#10" value="" x="18.415" y="11.43" smashed="yes" rot="MR0"/>
 <element name="U$18" library="output" package="#GND#4" value="" x="6.35" y="1.778" smashed="yes" rot="MR90"/>
-<element name="U$19" library="output" package="#3#3V#0" value="" x="8.89" y="1.778" smashed="yes" rot="MR90"/>
 <element name="U$20" library="output" package="#SDA#5" value="" x="11.43" y="1.778" smashed="yes" rot="MR90"/>
 <element name="U$21" library="output" package="#SCL#6" value="" x="13.97" y="1.778" smashed="yes" rot="MR90"/>
@@
 <element name="LOGO2" library="SparkFun-Aesthetics" package="SFE_LOGO_NAME_FLAME_.1" value="SFE_LOGO_NAME_FLAME.1_INCH" x="12.7" y="21.336" smashed="yes"/>
 <element name="LOGO4" library="SparkFun-Aesthetics" package="SFE_LOGO_NAME_FLAME_.1" value="SFE_LOGO_NAME_FLAME.1_INCH" x="12.7" y="21.336" smashed="yes" rot="MR0"/>
+<element name="U$3" library="output" package="#3V3#0" value="" x="8.89" y="1.778" smashed="yes" rot="MR90"/>
+<element name="U$2" library="output" package="VERSION_C0" value="" x="12.7" y="13.97" smashed="yes"/>
 </elements>
 <signals>
