File: Hardware/Qwiic_RFID_Tag.sch (EAGLE design)
At the start: 27 parts, among them J1 Qwiic, J2 Qwiic, U1 ST25DV64KC

Commit message: v10 Updates
Remove A and C versions, moving forward with B
Reorganize hardware folder
Rename coil library to match SFE library naming
Bump version number to v10
Smash power symbols to get vector font
Parts:
- removed H1, H2: STAND-OFF, SparkFun-Hardware:STAND-OFF
- L1: value PCB_COIL_4UH_A -> PCB_COIL_4UH_B; device QWIIC_RFID_TAG_COILS:PCB_COIL_4UH_A -> QWIIC_RFID_TAG_COILS:PCB_COIL_4UH_B
Connections:
- net 3.3V: now also R3.2; no longer JP3.2
- net GND: now also JP3.1; no longer D1.C
- net N$1: now also D1.C, JP3.2; no longer JP3.1, R3.2
Other:
- note added: "v10"
- note removed: "v03"
- moved on the sheet: D1, JP3, R3

Commit message: Add input voltage range
Other:
- note added: "Input voltage range: 1.8V - 5.5V"
Changed lines of the file:
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@@
 0x51 - RF Switch Off
 0x55 - RF Switch On</text>
+<text x="35.56" y="156.21" size="1.27" layer="97" font="vector">Input voltage range:
+1.8V - 5.5V</text>
 </plain>
 <instances>

Commit message: Bump version number to v11 and repanelize
Panelizer didn't work correctly on v10, none of the pads had nets assigned to them, so the GND polygon didn't connect to any GND pads. Repanlizing seems to fix it? Idk, it's whacky.
Other:
- note added: "v11"
- note removed: "v10"
Changed lines of the file:
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@@
 5.6 pF is the initial calculated value.</text>
 <wire x1="147.32" y1="50.8" x2="147.32" y2="35.56" width="0.2032" layer="97" style="longdash"/>
-<text x="241.3" y="7.62" size="2.54" layer="94" font="vector" align="center">v10</text>
+<text x="241.3" y="7.62" size="2.54" layer="94" font="vector" align="center">v11</text>
 <text x="180.34" y="12.7" size="2.54" layer="94" font="vector" align="center">Ricardo Ramos</text>
 <text x="167.64" y="7.62" size="2.54" layer="94" font="vector" align="center">Revised by:  Dryw Wade</text>

Commit message: Remove library file
Part is in SFE Eagle library, update part in design
Parts:
- L1: value PCB_COIL_4UH_B -> PCB_4UH_INDUCTOR-1X0.5; device QWIIC_RFID_TAG_COILS:PCB_COIL_4UH_B -> SparkFun-Coils:PCB_4UH_INDUCTOR-1X0.5
Changed lines of the file:
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@@
 <part name="J1" library="SparkFun-Connectors" deviceset="QWIIC_CONNECTOR" device="JS-1MM" value="Qwiic"/>
 <part name="J2" library="SparkFun-Connectors" deviceset="QWIIC_CONNECTOR" device="JS-1MM" value="Qwiic"/>
-<part name="L1" library="QWIIC_RFID_TAG_COILS" deviceset="PCB_COIL_4UH" device="_B" value="PCB_COIL_4UH_B"/>
+<part name="L1" library="SparkFun-Coils" deviceset="PCB_4UH_INDUCTOR" device="-1X0.5" value="PCB_4UH_INDUCTOR-1X0.5"/>
 <part name="C2" library="SparkFun-Capacitors" deviceset="4.7PF" device="-0603-50V-5%" value="4.7pF"/>
 <part name="GND5" library="SparkFun-PowerSymbols" deviceset="GND" device=""/>
